File: pcb-gary-ext/pcb-gary-ext.kicad_pcb (KiCad board)
At the start: 2 copper layers, 74 x 22 mm, 12 parts, among them J1 CONN_02X04, J2 CONN_01X02, U1 GARY, U2 GARY, U3 GAL16V8

Commit message: Updated schmatic.
Other:
- board text added: "CDAC"
- board text added: "OVL"
- board text added: "RST"
Changed lines of the file:
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@@
   (general
     (thickness 1.6)
-    (drawings 15)
+    (drawings 34)
     (tracks 168)
     (zones 0)
@@
     (pad_to_mask_clearance 0.051)
     (solder_mask_min_width 0.25)
-    (aux_axis_origin 0 0)
+    (aux_axis_origin 95 99)
     (visible_elements FFFFFF7F)
     (pcbplotparams
@@
       (viasonmask false)
       (mode 1)
-      (useauxorigin false)
+      (useauxorigin true)
       (hpglpennumber 1)
       (hpglpenspeed 20)
@@
       (outputformat 1)
       (mirror false)
-      (drillshape 1)
+      (drillshape 0)
       (scaleselection 1)
-      (outputdirectory ""))
+      (outputdirectory "Gerber"))
   )
   (net 0 "")
@@
     )
   )
+  (gr_line (start 149.606 98.044) (end 149.86 97.79) (layer F.SilkS) (width 0.12))
+  (gr_line (start 147.32 97.79) (end 147.574 98.044) (layer F.SilkS) (width 0.12))
+  (gr_line (start 149.86 97.79) (end 149.86 96.012) (layer F.SilkS) (width 0.12))
+  (gr_line (start 147.574 98.044) (end 149.606 98.044) (layer F.SilkS) (width 0.12))
+  (gr_text RST (at 148.59 98.552) (layer F.SilkS)
+    (effects (font (size 0.6 0.8) (thickness 0.15)))
+  )
+  (gr_line (start 147.32 96.012) (end 147.32 97.79) (layer F.SilkS) (width 0.12))
+  (gr_text CDAC (at 110.49 98.552) (layer F.SilkS)
+    (effects (font (size 0.6 0.8) (thickness 0.15)))
+  )
+  (gr_line (start 109.22 97.79) (end 109.474 98.044) (layer F.SilkS) (width 0.12))
+  (gr_line (start 111.506 98.044) (end 111.76 97.79) (layer F.SilkS) (width 0.12))
+  (gr_text OVL (at 120.65 98.552) (layer F.SilkS)
+    (effects (font (size 0.6 0.8) (thickness 0.15)))
+  )
+  (gr_line (start 121.92 97.79) (end 121.92 96.012) (layer F.SilkS) (width 0.12))
+  (gr_line (start 121.666 98.044) (end 121.92 97.79) (layer F.SilkS) (width 0.12))
+  (gr_line (start 119.634 98.044) (end 121.666 98.044) (layer F.SilkS) (width 0.12))
+  (gr_line (start 119.38 97.79) (end 119.634 98.044) (layer F.SilkS) (width 0.12))
+  (gr_line (start 119.38 96.012) (end 119.38 97.79) (layer F.SilkS) (width 0.12))
+  (gr_line (start 114.3 96.012) (end 119.38 96.012) (layer F.SilkS) (width 0.12))
+  (gr_line (start 111.76 97.79) (end 111.76 96.012) (layer F.SilkS) (width 0.12))
+  (gr_line (start 109.474 98.044) (end 111.506 98.044) (layer F.SilkS) (width 0.12))
+  (gr_line (start 109.22 96.012) (end 109.22 97.79) (layer F.SilkS) (width 0.12))
   (gr_text "GAL (T4)" (at 132.08 88.392) (layer F.SilkS)
     (effects (font (size 1 1) (thickness 0.15)))
