File: pcb-trapdoor/trapdoor.kicad_pcb (KiCad board)
At the start: 2 copper layers, 41 x 74 mm, 47 parts, among them J1 TRAPDOOR-CONNECTOR, J2 TEST_1P, J3 CONN_01X03, J4 CONN_01X02, U1 DRAM-1Mx16-SOJ-42, U5 GAL16V8, U6 74HC04, U7 MSM6242, Y1 32,768kHz

Commit message: PCBs hinzugefügt.
Routing:
- net /XA4: track 12.3 -> 8.72 mm
- net /XA2: track 5.16 -> 8.70 mm

Commit message: Update PCB für Trapdoor.
Parts:
- BT1: footprint Battery_Holders:Keystone_104_1x23mm-CoinCell -> Conn2:BAT-CR2032
- moved BT1 7.25 mm to (84.8, 96.8)
- moved C7 3.34 mm to (71.4, 76.2), turned to 180 degrees
- moved J4 2.79 mm to (63.5, 114.3)
- moved Y1 2.53 mm to (72.3, 86.3)
- moved C8 2.38 mm to (70.4, 88.9)
- moved C9 2.38 mm to (72.4, 88.9)
- moved R6 2.09 mm to (61.7, 121.4)
- moved R10 2.09 mm to (61.7, 117.3)
- moved R2 2.09 mm to (61.7, 125.5)
- moved R4 2.09 mm to (61.7, 123.4)
- moved R8 2.09 mm to (61.7, 119.4)
- moved R19 1.93 mm to (71.4, 93.5)
- moved SJ2 1.81 mm to (76.5, 118.8)
- moved SJ3 1.67 mm to (78.0, 118.9)
- moved SJ1 0.82 mm to (79.5, 118.9)
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Connections:
- R10 pad 1: /A4 -> /A6
- R2 pad 1: /A0 -> /A1
- R3 pad 1: /A1 -> /A0
- R4 pad 1: /A8 -> /A3
- R6 pad 1: /A7 -> /A5
- R7 pad 1: /A3 -> /A4
- R8 pad 1: /A6 -> /A7
- R9 pad 1: /A5 -> /A8
- U1 pad 18: /A1 -> /A2
- U1 pad 19: /A2 -> /A4
- U1 pad 20: /A3 -> /A8
- U1 pad 23: /A4 -> /A9
- U1 pad 24: /A5 -> /A6
- U1 pad 25: /A6 -> /A7
- U1 pad 26: /A7 -> /A5
- U1 pad 27: /A8 -> /A3
- U1 pad 28: /A9 -> /A1
- U5 pad 12: /~CASL -> (no net)
- U5 pad 13: /~CASU -> (no net)
- U5 pad 14: /~RAS -> /~CASL
- U5 pad 15: /A9 -> /~CASU
- U5 pad 16: (no net) -> /~RAS
- U5 pad 17: (no net) -> /A9
- U5 pad 7: /~CASL_IN -> /~CASU_IN
- U5 pad 8: /~CASU_IN -> /~CASL_IN
Routing:
- net +5V: track 233.7 -> 205.4 mm
- net /A8: track 24.2 -> 37.1 mm
- net /A3: track 35.1 -> 23.8 mm
- net /~RAS: track 28.2 -> 37.3 mm, vias 2 -> 0
- net /A1: track 29.8 -> 20.9 mm
- net /A9: track 20.1 -> 12.9 mm, vias 2 -> 0
- net Net-(BT1-Pad1): track 19.6 -> 13.3 mm
- net Net-(J1-Pad30): track 10.4 -> 16.1 mm
- net /~CASL: track 19.7 -> 14.4 mm, vias 4 -> 2
- net /A0: track 33.8 -> 28.9 mm
- net /~CASU_IN: track 16.4 -> 20.1 mm
- net /A6: track 29.2 -> 32.6 mm
- net Net-(C7-Pad2): track 27.3 -> 24.1 mm
- net /SEL0: track 30.1 -> 33.1 mm
- net /A7: track 26.6 -> 29.6 mm
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Other:
- board size 41 x 74 mm -> 40 x 74 mm
- board text added: "Trapdoor Expansion jmA500 2020 v1.0 - Thanks to Individual Computers GmbH"
- board text removed: "Trapdoor Expansion jmA500 2020 v 1.0 Thanks to Individual Computers GmbH"

Commit message: Updated schmatic.
Parts:
- moved J3 5.08 mm to (70.6, 108.2), turned to 90 degrees
Routing:
- net /SEL1: track 28.2 -> 26.4 mm
- net Net-(U5-Pad18): track 30.6 -> 29.7 mm
- net /XD1: track 19.6 -> 18.9 mm
- net /SEL0: track 33.1 -> 33.8 mm
- net Net-(J1-Pad37): track 6.53 -> 5.83 mm
