File: pcb-trapdoor/trapdoor.sch (KiCad schematic (older format))
At the start: 47 parts, among them J1 TRAPDOOR-CONNECTOR, J2 TEST_1P, J3 CONN_01X03, J4 CONN_01X02, U1 DRAM-1Mx16-SOJ-42, U5 GAL16V8, U6 74HC04, U7 MSM6242, Y1 32,768kHz

Commit message: Update PCB für Trapdoor.
Parts:
- BT1: footprint Battery_Holders:Keystone_104_1x23mm-CoinCell -> Conn2:BAT-CR2032
Connections:
- net A0: now also R3.1; no longer R2.1
- net A1: now also R2.1, U1.28 (A9); no longer R3.1, U1.18 (A1)
- net A2: now also U1.18 (A1); no longer U1.19 (A2)
- net A3: now also R4.1, U1.27 (A8); no longer R7.1, U1.20 (A3)
- net A4: now also R7.1, U1.19 (A2); no longer R10.1, U1.23 (A4)
- net A5: now also R6.1, U1.26 (A7); no longer R9.1, U1.24 (A5)
- net A6: now also R10.1, U1.24 (A5); no longer R8.1, U1.25 (A6)
- net A7: now also R8.1, U1.25 (A6); no longer R6.1, U1.26 (A7)
- net A8: now also R9.1, U1.20 (A3); no longer R4.1, U1.27 (A8)
- net A9: now also U1.23 (A4), U5.17 (I03); no longer U1.28 (A9), U5.15 (IO5)
- net ~CASL: now also U5.14 (IO6); no longer U5.12 (IO8)
- net ~CASL_IN: now also U5.8 (I8); no longer U5.7 (I7)
- net ~CASU: now also U5.15 (IO5); no longer U5.13 (IO7)
- net ~CASU_IN: now also U5.7 (I7); no longer U5.8 (I8)
- net ~RAS: now also U5.16 (IO4); no longer U5.14 (IO6)
Other:
- moved on the sheet: R16
Changed lines of the file:
@@
 F 0 "BT1" H 6450 6750 50  0000 L CNN
 F 1 "CR2032 Battery Holder" H 6500 7150 50  0000 L CNN
-F 2 "Battery_Holders:Keystone_104_1x23mm-CoinCell" V 6400 6860 50  0001 C CNN
+F 2 "Conn2:BAT-CR2032" V 6400 6860 50  0001 C CNN
 F 3 "~" V 6400 6860 50  0001 C CNN
 	1    6400 6800
@@
 A0
 Text Label 4600 1400 0    50   ~ 0
-A1
+A2
+Text Label 4600 2100 0    50   ~ 0
+A3
 Text Label 4600 1500 0    50   ~ 0
-A2
+A4
+Text Label 4600 2000 0    50   ~ 0
+A5
+Text Label 4600 1800 0    50   ~ 0
+A6
+Text Label 4600 1900 0    50   ~ 0
+A7
 Text Label 4600 1600 0    50   ~ 0
-A3
-Text Label 4600 1700 0    50   ~ 0
-A4
-Text Label 4600 1800 0    50   ~ 0
-A5
-Text Label 4600 1900 0    50   ~ 0
-A6
-Text Label 4600 2000 0    50   ~ 0
-A7
-Text Label 4600 2100 0    50   ~ 0
 A8
-Text Label 4600 2200 0    50   ~ 0
-A9
 Wire Wire Line
 	4600 2500 4850 2500
@@
 Wire Wire Line
 	2100 4000 2550 4000
+Text Label 2550 3200 2    50   ~ 0
+A0
 Text Label 2550 3300 2    50   ~ 0
-A0
-Text Label 2550 3200 2    50   ~ 0
 A1
 Text Label 2550 3400 2    50   ~ 0
 A2
+Text Label 2550 3500 2    50   ~ 0
+A3
 Text Label 2550 3600 2    50   ~ 0
-A3
+A4
+Text Label 2550 3700 2    50   ~ 0
+A5
 Text Label 2550 3800 2    50   ~ 0
-A4
+A6
+Text Label 2550 3900 2    50   ~ 0
+A7
 Text Label 2550 4000 2    50   ~ 0
-A5
-Text Label 2550 3900 2    50   ~ 0
-A6
-Text Label 2550 3700 2    50   ~ 0
-A7
-Text Label 2550 3500 2    50   ~ 0
 A8
 Entry Wire Line
@@
 Wire Wire Line
 	6950 2300 7250 2300
-NoConn ~ 8250 1700
-NoConn ~ 8250 1800
+NoConn ~ 8250 2100
+NoConn ~ 8250 2200
 Text Label 6950 1900 0    50   ~ 0
 ~RAS0_IN
 Text Label 6950 2000 0    50   ~ 0
 ~RAS1_IN
+Text Label 6950 2200 0    50   ~ 0
+~CASL_IN
 Text Label 6950 2100 0    50   ~ 0
-~CASL_IN
-Text Label 6950 2200 0    50   ~ 0
 ~CASU_IN
 $Comp
@@
 	7200 2400 7200 2450
 Wire Wire Line
+	8250 1700 8500 1700
+Wire Wire Line
+	8250 1800 8500 1800
+Wire Wire Line
+	8250 2000 8500 2000
+Wire Wire Line
 	8250 1900 8500 1900
-Wire Wire Line
-	8250 2000 8500 2000
-Wire Wire Line
-	8250 2100 8500 2100
-Wire Wire Line
-	8250 2200 8500 2200
+Text Label 8500 1700 2    50   ~ 0
+A9
+Text Label 8500 2000 2    50   ~ 0
+~CASL
 Text Label 8500 1900 2    50   ~ 0
-A9
-Text Label 8500 2200 2    50   ~ 0
-~CASL
-Text Label 8500 2100 2    50   ~ 0
 ~CASU
-Text Label 8500 2000 2    50   ~ 0
+Text Label 8500 1800 2    50   ~ 0
 ~RAS
 $Comp
@@
 L Device:R R16
 U 1 1 5EE812E0
-P 4300 1950
-F 0 "R16" H 4369 1904 50  0000 L CNN
-F 1 "4k7" H 4369 1995 50  0000 L CNN
-F 2 "discrete:R_0805" V 4230 1950 50  0001 C CNN
-F 3 "~" H 4300 1950 50  0001 C CNN
-	1    4300 1950
+P 4250 1500
+F 0 "R16" H 4319 1454 50  0000 L CNN
+F 1 "4k7" H 4319 1545 50  0000 L CNN
+F 2 "discrete:R_0805" V 4180 1500 50  0001 C CNN
+F 3 "~" H 4250 1500 50  0001 C CNN
+	1    4250 1500
 	-1   0    0    1
 $EndComp
 Wire Wire Line
-	4600 2200 4600 2250
-Wire Wire Line
-	4600 2250 4300 2250
-Text Label 4150 2250 0    50   ~ 0
+	4500 1800 4250 1800
+Text Label 4600 1700 0    50   ~ 0
 A9
 Wire Wire Line
-	4300 2100 4300 2250
-Connection ~ 4300 2250
-Wire Wire Line
-	4300 2250 4150 2250
+	4250 1650 4250 1800
+Connection ~ 4250 1800
+Wire Wire Line
+	4250 1800 4100 1800
 $Comp
 L power-own:+5V #PWR0112
 U 1 1 5EEC7B97
-P 4300 1800
-F 0 "#PWR0112" H 4300 1650 50  0001 C CNN
-F 1 "+5V" H 4300 1973 50  0000 C CNN
-F 2 "" H 4300 1800 50  0001 C CNN
-F 3 "" H 4300 1800 50  0001 C CNN
-	1    4300 1800
+P 4250 1350
+F 0 "#PWR0112" H 4250 1200 50  0001 C CNN
+F 1 "+5V" H 4250 1523 50  0000 C CNN
+F 2 "" H 4250 1350 50  0001 C CNN
+F 3 "" H 4250 1350 50  0001 C CNN
+	1    4250 1350
 	1    0    0    -1
 $EndComp
@@
 Wire Notes Line
 	8150 3100 8150 6500
+Text Label 4100 1800 0    50   ~ 0
+A9
+Text Label 4600 2200 0    50   ~ 0
+A1
+Entry Wire Line
+	4500 2300 4600 2200
 Wire Wire Line
 	2100 4700 3000 4700

Commit message: Updated schmatic.
Other:
- note removed: "Lower Byte"
Changed lines of the file:
@@
 	2550 4800 2650 4700
 Wire Bus Line
-	4500 3250 3300 3250
+	4500 2950 4450 3000
 NoConn ~ 1500 4900
 Entry Wire Line
@@
 	2650 3050 2700 3000
 Wire Bus Line
-	2700 3000 3200 3000
-Wire Bus Line
-	3200 3000 3250 3050
-Wire Bus Line
 	3950 800  4000 750
-Wire Bus Line
-	4000 750  6200 750
-Wire Bus Line
-	3300 3250 3250 3200
-Wire Bus Line
-	3250 3050 3250 3200
 Text Notes 3650 7650 0    100  ~ 0
 Optional: Clock
-Text Notes 6500 650  0    100  ~ 0
-Lower Byte
 Text Notes 2250 700  0    50   ~ 0
 Pull-Ups on Data Lines \nare optional
@@
 Entry Wire Line
 	4500 2300 4600 2200
+Wire Bus Line
+	2700 3000 4450 3000
+Wire Bus Line
+	6200 800  6150 750
+Wire Bus Line
+	6150 750  4000 750
 Wire Wire Line
 	2100 4700 3000 4700
@@
 	2750 5900 2750 7250
 Wire Bus Line
-	4500 1400 4500 3250
+	4500 1400 4500 2950
 Wire Bus Line
 	3950 800  3950 2800
 Wire Bus Line
-	6200 750  6200 2800
+	6200 800  6200 2800
 $EndSCHEMATC
